Commit message: Supports both cameras

File: softdrone_core/urdf/drone.urdf.xacro (robot description, xacro)
@@ -3,21 +3,7 @@
 <robot name="softdrone" xmlns:xacro="http://www.ros.org/wiki/xacro">
   <xacro:property name="PI" value="3.1415926535897931" />
-  <xacro:property name="camera_offset_len" value="0.1" />
-  <xacro:property name="camera_offset_ver" value="0.0" />
-  <!-- +- 35 degrees -->
-  <!--
-  <xacro:property name="pan_range" value="0.6108652381980153" />
-  <xacro:property name="pan_vel" value="2.0" />
-  -->
-  <!-- +- 35 degrees -->
-  <!--
-  <xacro:property name="tilt_range" value="0.6108652381980153" />
-  <xacro:property name="tilt_vel" value="2.0" />
-  <xacro:property name="joint_effort" value="50" />
-  -->
-  <!--link name="root_link"></link-->
     <link name="base_link">
      <visual>
-        <origin xyz="0 0 0" rpy="0 0 ${PI}" />
+        <origin xyz="0.275 0.12 0.05" rpy="0 0 ${PI}" />
         <geometry>
           <mesh scale=".001 .001 .001" filename="package://softdrone_core/meshes/drone_mesh_v27.stl"/>
@@ -25,11 +11,15 @@
      </visual>
     </link>
-    <link name="camera_pose_frame"></link>
-    <joint name="base_link_joint" type="fixed">
-      <origin xyz="0 0 0" rpy="0 0.785 0" />
+    <link name="nav_cam_pose_frame"></link>
+    <link name="target_cam_link"></link>
+    <joint name="base_link_to_nav_cam" type="fixed">
+      <origin xyz="-0.08 0 0" rpy="0 0.785 ${PI}" />
       <parent link="base_link"/>
-      <child link="camera_pose_frame" />
+      <child link="nav_cam_pose_frame" />
     </joint>
-  <!-- [nice to have] -->
-  <!-- xacro:include filename="bebop.gazebo" /-->
+    <joint name="base_link_to_target_cam" type="fixed">
+      <origin xyz="0.08 0 0" rpy="0 0.785 0" />
+      <parent link="base_link"/>
+      <child link="target_cam_link" />
+    </joint>
 </robot>

Commit message: Updated full_drone.launch for new drone

File: softdrone_core/urdf/drone.urdf.xacro (robot description, xacro)
@@ -14,5 +14,5 @@
     <link name="target_cam_link"></link>
     <joint name="base_link_to_nav_cam" type="fixed">
-      <origin xyz="-0.08 0 0" rpy="0 0.785 ${PI}" />
+      <origin xyz="-0.08 0 0" rpy="0 0.611 ${PI}" />
       <parent link="base_link"/>
       <child link="nav_cam_pose_frame" />

Commit message: Updates to run pose detection better on Drone
* Reduced trajectory replanning rate for computational burden reasons
* Updated keypoint detector model
* Made covariance of pose estimate a parameter instead of hard-coded
* Made plant covariance in EKF a parameter
* Updated launch files for drone testing

File: softdrone_core/urdf/drone.urdf.xacro (robot description, xacro)
@@ -19,5 +19,5 @@
     </joint>
     <joint name="base_link_to_target_cam" type="fixed">
-      <origin xyz="0.08 0 0" rpy="0 0.785 0" />
+      <origin xyz="0.08 0 0" rpy="0 0.611 0" />
       <parent link="base_link"/>
       <child link="target_cam_link" />

Commit message: urdf update for straight camera and waiting for new trajectory at hover

File: softdrone_core/urdf/drone.urdf.xacro (robot description, xacro)
@@ -14,5 +14,5 @@
     <link name="target_cam_link"></link>
     <joint name="base_link_to_nav_cam" type="fixed">
-      <origin xyz="-0.08 0 0" rpy="0 0.611 ${PI}" />
+      <origin xyz="-0.08 0 0" rpy="0 0 ${PI}" />
       <parent link="base_link"/>
       <child link="nav_cam_pose_frame" />

Commit message: Grasp w/ new gripper 5/31

File: softdrone_core/urdf/drone.urdf.xacro (robot description, xacro)
@@ -14,5 +14,5 @@
     <link name="target_cam_link"></link>
     <joint name="base_link_to_nav_cam" type="fixed">
-      <origin xyz="-0.08 0 0" rpy="0 0 ${PI}" />
+      <origin xyz="-0.08 0 0" rpy="0 0.611 ${PI}" />
       <parent link="base_link"/>
       <child link="nav_cam_pose_frame" />
